File: playground/LEDx16Module/kicad_project/LEDx16_board.kicad_pcb (KiCad board)
At the start: 2 copper layers, 45.7 x 31.8 mm, 36 parts, among them P1 CONN_01X05, U1 74HC595, U2 74HC595

Commit message: [LEDx16Module] notes after fab and build
Connections:
- U1 pad 13: Net-(U1-Pad13) -> GND
- U2 pad 13: Net-(U2-Pad13) -> GND
Routing:
- net GND: track 43.5 -> 53.8 mm, vias 3 -> 4
- net VCC: track 158.8 -> 159.3 mm
Other:
- board text added: "CLK"
- board text added: "DATA"
- board text added: "DS"
- board text added: "GND"
- board text added: "LATCH"
- board text added: "LEDx16 Board 1.0.1"
- board text added: "SH_CP"
- board text added: "ST_CP"
- board text added: "VCC"
- board text removed: "LEDx16 Board 1.0.0"
