File: playground/LEDx16Module/kicad_project/LEDx16_board.sch (KiCad schematic (older format))
At the start: 36 parts, among them P1 CONN_01X05, U1 74HC595, U2 74HC595

Commit message: [LEDx16Module] notes after fab and build
Connections:
- net GND: now also U1.13 (G), U2.13 (G)
- no-connect marks 3 -> 1
Changed lines of the file:
@@
 Title "16 LED board"
 Date "2016-01-26"
-Rev "1.0.0"
+Rev "1.0.1"
 Comp "github.com/tardate/LittleArduinoProjects"
 Comment1 ""
@@
 Wire Wire Line
 	1200 1600 1300 1600
-NoConn ~ 1300 1900
 Text Label 2700 2200 0    60   ~ 0
 CARRY
@@
 Wire Wire Line
 	4000 1600 4100 1600
-NoConn ~ 4100 1900
 NoConn ~ 5500 2200
 Wire Notes Line
@@
 Wire Notes Line
 	900  5300 900  1100
+$Comp
+L GND #PWR011
+U 1 1 574154D0
+P 1300 1900
+F 0 "#PWR011" H 1300 1650 50  0001 C CNN
+F 1 "GND" H 1300 1750 50  0000 C CNN
+F 2 "" H 1300 1900 50  0000 C CNN
+F 3 "" H 1300 1900 50  0000 C CNN
+	1    1300 1900
+	1    0    0    -1
+$EndComp
+$Comp
+L GND #PWR012
+U 1 1 57415675
+P 4100 1900
+F 0 "#PWR012" H 4100 1650 50  0001 C CNN
+F 1 "GND" H 4100 1750 50  0000 C CNN
+F 2 "" H 4100 1900 50  0000 C CNN
+F 3 "" H 4100 1900 50  0000 C CNN
+	1    4100 1900
+	1    0    0    -1
+$EndComp
 $EndSCHEMATC
